File: PCB/Driver.kicad_pcb (KiCad board)
At the start: 2 copper layers, 62 x 50 mm, 50 parts, among them IC1 ESP32-PICO-V3, IC2 LMR36506, IC3 MA702GQ-P, IC4 SN65HVD230QDRG4, J1 XT30PB, U1 DRV8316R

Commit message: Update to v0.21
Parts:
- removed REF**: KiCad-Logo2_5mm_SilkScreen, Symbol:KiCad-Logo2_5mm_SilkScreen
- added G***: LOGO, DriverParts:KiCad, F.Cu at (159.3, 115.5)
- moved G*** 10.4 mm to (159.0, 108.7)
- moved JP1 4.36 mm to (156.6, 107.4)
Routing:
- net Net-(CAN1-Pad2): track 40.6 -> 38.4 mm
- net Net-(JP1-Pad1): track 20.5 -> 21.3 mm
- net GND: vias 82 -> 79
Other:
- board text added: "Stealth Controller v0.21"
- board text added: "TWAI"
- board text added: "TWAI 120Ω"
- board text removed: "CAN"
- board text removed: "CAN 120Ω"
- board text removed: "v0.21"
