File: PCB/Driver.sch (KiCad schematic (older format))
At the start: 47 parts, among them IC1 ESP32-PICO-V3, IC2 LMR36506, IC3 MA702GQ-P, IC4 SN65HVD230QDRG4, J1 XT30PB, U1 DRV8316R

Commit message: Update to v0.21
Parts:
- TWAI1: renamed from CAN1; value CAN -> TWAI
- TWAI2: renamed from CAN2; value CAN -> TWAI
Other:
- note added: "TWAI"
- note removed: "CAN"
Changed lines of the file:
@@
 encoding utf-8
 Sheet 1 1
-Title "Driver Board (DRV8316 + ESP32 + MA702 + CAN)"
+Title "Driver Board (DRV8316 + ESP32 + MA702 + TWAI)"
 Date "2021-04-09"
 Rev "0.2"
@@
 Magnetic Encoder
 Text Notes 8900 5050 0    79   ~ 16
-CAN
+TWAI
 Text Notes 2400 5050 0    79   ~ 16
 Power
@@
 $EndComp
 $Comp
-L DriverParts:S3B-ZR-SM4A-TF CAN2
+L DriverParts:S3B-ZR-SM4A-TF TWAI2
 U 1 1 602AD11B
 P 10500 5750
-F 0 "CAN2" H 10730 5696 50  0001 L CNN
-F 1 "CAN" H 10730 5605 50  0000 L CNN
+F 0 "TWAI2" H 10730 5696 50  0001 L CNN
+F 1 "TWAI" H 10730 5605 50  0000 L CNN
 F 2 "DriverParts:SHDR3W50P0X150" H 10500 5750 50  0001 L BNN
 F 3 "S3B-ZR-SM4A-TF" H 10500 5750 50  0001 L BNN
@@
 	10300 5400 10250 5400
 $Comp
-L DriverParts:S3B-ZR-SM4A-TF CAN1
+L DriverParts:S3B-ZR-SM4A-TF TWAI1
 U 1 1 6058F40E
 P 10500 5300
-F 0 "CAN1" H 10730 5246 50  0001 L CNN
-F 1 "CAN" H 10730 5155 50  0000 L CNN
+F 0 "TWAI1" H 10730 5246 50  0001 L CNN
+F 1 "TWAI" H 10730 5155 50  0000 L CNN
 F 2 "DriverParts:SHDR3W50P0X150" H 10500 5300 50  0001 L BNN
 F 3 "S3B-ZR-SM4A-TF" H 10500 5300 50  0001 L BNN
